File: kicad/ez-dipole/ez-dipole.kicad_sch (KiCad schematic)
At the start: 3 parts, among them J1 Conn_Coaxial

Commit message: Increased slot length outside of board outline and adapted SMA footprint to allow also smaller SMA connectors
Parts:
- J1: footprint Connector_Coaxial:SMA_Amphenol_132289_EdgeMount -> ez-dipole:SMA_Amphenol_132289_EdgeMount
Changed lines of the file:
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@@
     (property "Reference" "J1" (id 0) (at 99.06 80.9626 0))
     (property "Value" "Conn_Coaxial" (id 1) (at 101.6 80.9626 0))
-    (property "Footprint" "Connector_Coaxial:SMA_Amphenol_132289_EdgeMount" (id 2) (at 106.68 81.28 0)
+    (property "Footprint" "ez-dipole:SMA_Amphenol_132289_EdgeMount" (id 2) (at 106.68 81.28 0)
       (effects (font (size 1.27 1.27)) hide)
     )
@@
     )
     (path "/d385ebb9-fe43-4fe3-ae5a-b83665559f7f"
-      (reference "J1") (unit 1) (value "Conn_Coaxial") (footprint "Connector_Coaxial:SMA_Amphenol_132289_EdgeMount")
+      (reference "J1") (unit 1) (value "Conn_Coaxial") (footprint "ez-dipole:SMA_Amphenol_132289_EdgeMount")
     )
     (path "/c67cf94f-d750-45b8-b736-ef5a3f3d0d84"
